Commit message: Implementación de jointrajectory para movimientos suaves en el rviz

File: Nicolas_Tafur/install/robot/share/robot/urdf/robot.xacro (robot description, xacro)
@@ -1 +1,327 @@
-/home/richilzz/ros2_ws/src/git/Robotica-UAO-2025-3/Nicolas_Tafur/build/robot/urdf/robot.xacro
+<?xml version="1.0"?>
+<robot xmlns:xacro="http://www.ros.org/wiki/xacro"
+       name="simple_arm_3dof">
+  <!-- ============================= -->
+  <!--   LINK 0: Base vertical       -->
+  <!-- ============================= -->
+  <link name="estructurabasevertical">
+    <visual>
+      <origin xyz="0 0 0.18" rpy="0 0 0"/>
+      <geometry>
+        <box size="0.02 0.02 0.36"/>
+      </geometry>
+      <material name="gray">
+        <color rgba="0.5 0.5 0.5 1"/>
+      </material>
+    </visual>
+  </link>
+  <!-- ============================= -->
+  <!--   LINK 0.1: Base horizontal   -->
+  <!-- ============================= -->
+  <link name="estructurabasehorizontal">
+    <visual>
+      <geometry>
+        <box size="0.25 0.02 0.02"/>
+      </geometry>
+      <material name="gray">
+        <color rgba="0.5 0.5 0.5 1"/>
+      </material>
+    </visual>
+  </link>
+  <!-- ============================= -->
+  <!--   JOINT: Base fijo            -->
+  <!-- ============================= -->
+  <joint name="base_to_horizontal" type="fixed">
+    <parent link="estructurabasevertical"/>
+    <child  link="estructurabasehorizontal"/>
+    <origin xyz="0 0 0.36" rpy="0 0 0"/>
+  </joint>
+  <!-- ============================= -->
+  <!--   LINK: Hombro con dos dots   -->
+  <!-- ============================= -->
+  <link name="hombro">
+    <!-- Primera esfera -->
+    <visual>
+      <origin xyz=" 0 0 0" rpy="0 0 0"/>
+      <geometry>
+        <sphere radius="0.03"/>
+      </geometry>
+      <material name="gray">
+        <color rgba="0.5 0.5 0.5 1"/>
+      </material>
+    </visual>
+  </link>
+  <!-- ============================= -->
+  <!--   JOINT: Hombro → Primer brazo -->
+  <!-- ============================= -->
+  <joint name="joint1" type="revolute">
+    <parent link="estructurabasehorizontal"/>
+    <child  link="hombro"/>
+    <origin xyz="0.125 0 0" rpy="0 0 0"/>
+    <axis xyz="0 0 1"/>
+    <limit lower="-1.57" upper="1.57" effort="1.0" velocity="1.0"/>
+  </joint>
+  <!-- ============================= -->
+  <!--   LINK 1: Primer brazo        -->
+  <!-- ============================= -->
+  <link name="P1">
+    <visual>
+      <origin xyz="0 0 -0.025" rpy="0 0 0"/>
+      <geometry>
+        <box size="0.05 0.03 0.005"/>
+      </geometry>
+      <material name="gray">
+        <color rgba="0.5 0.5 0.5 1"/>
+      </material>
+    </visual>
+  </link>
+  <joint name="P1-2" type="fixed">
+    <parent link="P1"/>
+    <child  link="P2"/>
+    <origin xyz="0.025 0 -0.025" rpy="0 0 0"/>
+  </joint>
+  <joint name="P1-3" type="fixed">
+    <parent link="P1"/>
+    <child  link="P3"/>
+    <origin xyz="-0.025 0 -0.025" rpy="0 0 0"/>
+  </joint>
+  <link name="P2">
+    <visual>
+      <origin xyz="0 0 -0.05" rpy="0 0 0"/>
+      <geometry>
+        <box size="0.005 0.03 0.1"/>
+      </geometry>
+      <material name="gray">
+        <color rgba="0.5 0.5 0.5 1"/>
+      </material>
+    </visual>
+  </link>
+  <joint name="P2-4" type="fixed">
+    <parent link="P2"/>
+    <child  link="P4"/>
+    <origin xyz="-0.025 0 -0.105" rpy="0 0 0"/>
+  </joint>
+  <link name="P3">
+    <visual>
+      <origin xyz="0 0 -0.05" rpy="0 0 0"/>
+      <geometry>
+        <box size="0.005 0.03 0.1"/>
+      </geometry>
+      <material name="gray">
+        <color rgba="0.5 0.5 0.5 1"/>
+      </material>
+    </visual>
+  </link>
+  <link name="P4">
+    <visual>
+      <origin xyz="0 0 0" rpy="0 0 0"/>
+      <geometry>
+        <box size="0.05 0.03 0.03"/>
+      </geometry>
+      <material name="gray">
+        <color rgba="0.5 0.5 0.5 1"/>
+      </material>
+    </visual>
+  </link>
+  <joint name="joint2" type="revolute">
+    <parent link="hombro"/>
+    <child  link="P1"/>
+    <origin xyz="0 0 0" rpy="0 0 0"/>
+    <axis xyz="1 0 0"/>
+    <limit lower="-1.57" upper="1.57" effort="1.0" velocity="1.0"/>
+  </joint>
+  <!-- ============================= -->
+  <!--   LINK 2: Segundo brazo       -->
+  <!-- ============================= -->
+  <joint name="joint3" type="revolute">
+    <parent link="P4"/>
+    <child  link="PP1"/>
+    <origin xyz="0 0 0" rpy="0 0 0"/>
+    <axis xyz="1 0 0"/>
+    <limit lower="-1.57" upper="1.57" effort="1.0" velocity="1.0"/>
+  </joint>
+  <joint name="joint4" type="fixed">
+    <parent link="PP1"/>
+    <child  link="PP2"/>
+    <origin xyz="0 0 0" rpy="0 0 0"/>
+  </joint>
+  <link name="PP1">
+    <visual>
+      <origin xyz="0.025 0 -0.05" rpy="0 0 0"/>
+      <geometry>
+        <box size="0.005 0.03 0.1"/>
+      </geometry>
+      <material name="gray">
+        <color rgba="0.5 0.5 0.5 1"/>
+      </material>
+    </visual>
+  </link>
+  <link name="PP2">
+    <visual>
+      <origin xyz="-0.025 0 -0.05" rpy="0 0 0"/>
+      <geometry>
+        <box size="0.005 0.03 0.1"/>
+      </geometry>
+      <material name="gray">
+        <color rgba="0.5 0.5 0.5 1"/>
+      </material>
+    </visual>
+  </link>
+  <joint name="joint5" type="fixed">
+    <parent link="PP1"/>
+    <child  link="PP3"/>
+    <origin xyz="0 0 -0.1" rpy="0 0 0"/>
+  </joint>
+  <link name="PP3">
+    <visual>
+      <origin xyz="0 0 0" rpy="0 0 0"/>
+      <geometry>
+        <box size="0.05 0.03 0.005"/>
+      </geometry>
+      <material name="gray">
+        <color rgba="0.5 0.5 0.5 1"/>
+      </material>
+    </visual>
+  </link>
+  <!-- ============================= -->
+  <!--   LINK 3: GRIPPER       -->
+  <joint name="joint6" type="fixed">
+    <parent link="PP3"/>
+    <child  link="muñeca"/>
+    <origin xyz="0 0 0" rpy="0 0 0"/>
+  </joint>
+  <joint name="joint_dedo11" type="fixed">  <!-- o revolute/continuous según necesites -->
+    <parent link="muñeca"/>
+    <child  link="dedo11"/>
+    <!-- Origin aquí posiciona el frame de dedo11 al final de muñeca -->
+    <origin xyz="0 0 -0.02" rpy="0 0 0"/>
+    <axis xyz="0 0 1"/>
+    <limit lower="-1.57" upper="1.57" effort="1.0" velocity="1.0"/>
+  </joint>
+  <link name="muñeca">
+    <visual>
+      <origin xyz=" 0 0 -0.015" rpy="0 0 0"/>
+      <geometry>
+        <sphere radius="0.02"/>
+      </geometry>
+      <material name="gray">
+        <color rgba="0.5 0.5 0.5 1"/>
+      </material>
+    </visual>
+  </link>
+  <link name="dedo11">
+    <visual>
+      <origin xyz="-0.02 0 -0.02" rpy="0 0.7854 0"/>
+      <geometry>
+        <box size="0.005 0.02 0.04"/>
+      </geometry>
+      <material name="gray">
+        <color rgba="0.5 0.5 0.5 1"/>
+      </material>
+    </visual>
+  </link>
+  <joint name="joint7" type="fixed">
+    <parent link="dedo11"/>
+    <child  link="dedo12"/>
+    <origin xyz="-0.035 0 -0.035" rpy="0 0 0"/>
+  </joint>
+  <link name="dedo12">
+    <visual>
+      <origin xyz="0 0 -0.02" rpy="0 0 0"/>
+      <geometry>
+        <box size="0.005 0.02 0.04"/>
+      </geometry>
+      <material name="gray">
+        <color rgba="0.5 0.5 0.5 1"/>
+      </material>
+    </visual>
+  </link>
+  <joint name="joint_dedo21" type="fixed">  <!-- o revolute/continuous según necesites -->
+    <parent link="muñeca"/>
+    <child  link="dedo21"/>
+    <!-- Origin aquí posiciona el frame de dedo11 al final de muñeca -->
+    <origin xyz="0 0 -0.02" rpy="0 0 0"/>
+    <axis xyz="0 1 0"/>
+    <limit lower="-1.57" upper="1.57" effort="1.0" velocity="1.0"/>
+  </joint>
+  <link name="dedo21">
+    <visual>
+      <origin xyz="0.02 0 -0.02" rpy="0 -0.7854 0"/>
+      <geometry>
+        <box size="0.005 0.02 0.04"/>
+      </geometry>
+      <material name="gray">
+        <color rgba="0.5 0.5 0.5 1"/>
+      </material>
+    </visual>
+  </link>
+  <joint name="joint8" type="fixed">
+    <parent link="dedo21"/>
+    <child  link="dedo22"/>
+    <origin xyz="0.035 0 -0.035" rpy="0 0 0"/>
+  </joint>
+  <link name="dedo22">
+    <visual>
+      <origin xyz="0 0 -0.02" rpy="0 0 0"/>
+      <geometry>
+        <box size="0.005 0.02 0.04"/>
+      </geometry>
+      <material name="gray">
+        <color rgba="0.5 0.5 0.5 1"/>
+      </material>
+    </visual>
+  </link>
+  <ros2_control name="SimpleArmSystem" type="system">
+    <hardware>
+      <!-- Para simulación -->
+      <plugin>fake_components/GenericSystem</plugin>
+      <param name="fake_sensor_commands">true</param>
+    </hardware>
+    <joint name="joint1">
+      <command_interface name="position"/>
+      <state_interface name="position"/>
+      <state_interface name="velocity"/>
+    </joint>
+    <joint name="joint2">
+      <command_interface name="position"/>
+      <state_interface name="position"/>
+      <state_interface name="velocity"/>
+    </joint>
+    <joint name="joint3">
+      <command_interface name="position"/>
+      <state_interface name="position"/>
+      <state_interface name="velocity"/>
+    </joint>
+  </ros2_control>
+  <!-- Transmissions -->
+  <transmission name="trans_joint1">
+    <type>transmission_interface/SimpleTransmission</type>
+    <joint name="joint1">
+      <hardwareInterface>hardware_interface/PositionJointInterface</hardwareInterface>
+    </joint>
+    <actuator name="motor1">
+      <hardwareInterface>hardware_interface/PositionJointInterface</hardwareInterface>
+      <mechanicalReduction>1</mechanicalReduction>
+    </actuator>
+  </transmission>
+  <transmission name="trans_joint2">
+    <type>transmission_interface/SimpleTransmission</type>
+    <joint name="joint2">
+      <hardwareInterface>hardware_interface/PositionJointInterface</hardwareInterface>
+    </joint>
+    <actuator name="motor2">
+      <hardwareInterface>hardware_interface/PositionJointInterface</hardwareInterface>
+      <mechanicalReduction>1</mechanicalReduction>
+    </actuator>
+  </transmission>
+  <transmission name="trans_joint3">
+    <type>transmission_interface/SimpleTransmission</type>
+    <joint name="joint3">
+      <hardwareInterface>hardware_interface/PositionJointInterface</hardwareInterface>
+    </joint>
+    <actuator name="motor3">
+      <hardwareInterface>hardware_interface/PositionJointInterface</hardwareInterface>
+      <mechanicalReduction>1</mechanicalReduction>
+    </actuator>
+  </transmission>
+</robot>
