Commit message: Correcciones del DH y otras cositas para que funcione bien

File: Nicolas_Tafur/install/robot/share/robot/urdf/URDF_LINKS.urdf (robot description, URDF)
Before this commit: robot URDF_LINKS, 7 links, 6 joints
Joints:
- joint joint1: axis 0 0 1 -> 0 0 -1
- joint joint2: axis 0 -1 0 -> 0 1 0
- joint joint6: axis 0 -1 0 -> 0 1 0
